File: pcb/pcb.kicad_pcb (KiCad board)
At the start: 4 copper layers, 109.5 x 152.4 mm, 127 parts, among them J1 USB_C_Receptacle_USB2.0, J2 JST - 1.00mm 4 Pin, J4 Conn_01x05, J5 Conn_01x05, J6 Conn_01x05, J7 Conn_01x05, SW72 SW_Push, SW73 SW_Push, U1 RP2040, U3 USBLC6-2SC6, U4 3.3V Fixed Regulator, U5 ZD25D40CNJGR, Y1 12MHz Crystal 3225

Commit message: added some more routing
Parts:
- removed J2: JST - 1.00mm 4 Pin, Connector_JST:JST_SH_SM04B-SRSS-TB_1x04-1MP_P1.00mm_Horizontal
- moved SW72 21.6 mm to (104.6, 139.1), turned to 180 degrees
- moved SW73 5.72 mm to (95.5, 139.1), turned to 180 degrees
- moved U3 2.09 mm to (111.9, 115.4)
- moved D25 1.65 mm to (122.2, 81.8)
- moved D26 1.65 mm to (103.2, 81.8)
- moved D31 1.65 mm to (122.2, 79.5)
- moved D32 1.65 mm to (103.2, 79.5)
- moved D28 1.65 mm to (65.0, 81.8)
- moved D34 1.65 mm to (65.0, 79.5)
- moved D27 1.65 mm to (84.1, 81.8)
- moved D33 1.65 mm to (84.1, 79.5)
- moved R5 1.46 mm to (115.5, 109.5)
- moved R4 0.71 mm to (112.4, 109.4), turned to 90 degrees
- turned F1 to 180 degrees
Connections:
- D1 pad 1: /Switch Matrix/COL0 -> GP4
- D10 pad 1: /Switch Matrix/COL3 -> GP7
- D11 pad 1: /Switch Matrix/COL4 -> GP8
- D12 pad 1: /Switch Matrix/COL5 -> GP9
- D13 pad 1: /Switch Matrix/COL0 -> GP4
- D14 pad 1: GP2 -> GP5
- D15 pad 1: GP3 -> GP6
- D16 pad 1: /Switch Matrix/COL3 -> GP7
- D17 pad 1: /Switch Matrix/COL4 -> GP8
- D18 pad 1: /Switch Matrix/COL5 -> GP9
- D19 pad 1: GP3 -> GP6
- D2 pad 1: GP2 -> GP5
- D20 pad 1: /Switch Matrix/COL3 -> GP7
- D21 pad 1: /Switch Matrix/COL4 -> GP8
- D22 pad 1: /Switch Matrix/COL5 -> GP9
- D3 pad 1: GP3 -> GP6
- D4 pad 1: /Switch Matrix/COL3 -> GP7
- D5 pad 1: /Switch Matrix/COL4 -> GP8
- D6 pad 1: /Switch Matrix/COL5 -> GP9
- D7 pad 1: /Switch Matrix/COL0 -> GP4
- D8 pad 1: GP2 -> GP5
- D9 pad 1: GP3 -> GP6
- J4 pad 1: /Switch Matrix/ROW0 -> GP10
- J4 pad 2: GP0 -> GP3
- J4 pad 3: GP1 -> GP2
- J4 pad 4: /Switch Matrix/ROW3 -> GP1
- J4 pad 5: /Switch Matrix/COL6 -> GP0
- J5 pad 1: /Switch Matrix/ROW0 -> /Switch Matrix/ROW0r
- J5 pad 2: GP0 -> /Switch Matrix/ROW1r
- J5 pad 3: GP1 -> /Switch Matrix/ROW2r
- J5 pad 4: /Switch Matrix/ROW3 -> /Switch Matrix/ROW3r
- J6 pad 1: /Switch Matrix/COL7 -> GP15
- J6 pad 2: /Switch Matrix/COL8 -> GP14
- J6 pad 3: /Switch Matrix/COL9 -> GP13
- J6 pad 4: /Switch Matrix/COL10 -> GP12
- J6 pad 5: /Switch Matrix/COL11 -> GP11
- MX1 pad 1: /Switch Matrix/ROW0 -> GP0
- MX10 pad 1: GP0 -> GP1
- MX11 pad 1: GP0 -> GP1
- MX12 pad 1: GP0 -> GP1
- MX13 pad 1: GP1 -> GP2
- MX14 pad 1: GP1 -> GP2
- MX15 pad 1: GP1 -> GP2
- MX16 pad 1: GP1 -> GP2
- MX17 pad 1: GP1 -> GP2
- MX18 pad 1: GP1 -> GP2
- MX19 pad 1: /Switch Matrix/ROW3 -> GP3
- MX2 pad 1: /Switch Matrix/ROW0 -> GP0
- MX20 pad 1: /Switch Matrix/ROW3 -> GP3
- MX21 pad 1: /Switch Matrix/ROW3 -> GP3
- MX22 pad 1: /Switch Matrix/ROW3 -> GP3
- MX3 pad 1: /Switch Matrix/ROW0 -> GP0
- MX4 pad 1: /Switch Matrix/ROW0 -> GP0
- MX45 pad 1: /Switch Matrix/ROW3 -> GP3
- MX5 pad 1: /Switch Matrix/ROW0 -> GP0
- MX6 pad 1: /Switch Matrix/ROW0 -> GP0
- MX7 pad 1: GP0 -> GP1
- MX8 pad 1: GP0 -> GP1
- MX9 pad 1: GP0 -> GP1
Routing:
- net /Switch Matrix/COL11r: track 0.00 -> 136.5 mm, vias 0 -> 2
- net /Switch Matrix/ROW2r: track 0.00 -> 124.1 mm, vias 0 -> 3
- net /Switch Matrix/ROW3r: track 0.00 -> 117.2 mm, vias 0 -> 2
- net /Switch Matrix/COL10r: track 0.00 -> 113.9 mm, vias 0 -> 2
- net /Switch Matrix/ROW0r: track 0.00 -> 112.3 mm
- net GP0: track 0.00 -> 112.3 mm
- net /Switch Matrix/COL9r: track 0.00 -> 103.7 mm, vias 0 -> 2
- net /Switch Matrix/ROW1r: track 0.00 -> 102.6 mm
- net GP2: track 0.00 -> 96.9 mm
- net GP1: track 0.00 -> 96.9 mm
- net /Switch Matrix/COL8r: track 0.00 -> 80.2 mm, vias 0 -> 2
- net GP3: track 0.00 -> 67.3 mm
- net /Switch Matrix/COL6r: track 0.00 -> 67.1 mm, vias 0 -> 2
- net /Switch Matrix/COL7r: track 0.00 -> 66.9 mm, vias 0 -> 4
- net /DP: track 0.00 -> 60.7 mm, vias 0 -> 2
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
Commit message: redid routing
Parts:
- removed J4, J5, J6, J7: Conn_01x05, Connector_JST:JST_GH_SM05B-GHS-TB_1x05-1MP_P1.25mm_Horizontal
- added H1: MountingHole, pcb:spacer_hole_4mm, F.Cu at (78.6, 121.4)
- added H2: MountingHole, pcb:spacer_hole_4mm, F.Cu at (92.9, 154.8)
- added H3: MountingHole, pcb:spacer_hole_4mm, F.Cu at (150.0, 159.5)
- added H4: MountingHole, pcb:spacer_hole_4mm, F.Cu at (131.0, 111.9)
- added H5: MountingHole, pcb:spacer_hole_4mm, F.Cu at (78.6, 78.6)
- added H6: MountingHole, pcb:spacer_hole_4mm, F.Cu at (92.9, 45.2)
- added H7: MountingHole, pcb:spacer_hole_4mm, F.Cu at (150.0, 40.5)
- added H8: MountingHole, pcb:spacer_hole_4mm, F.Cu at (131.0, 88.1)
- added J2: Conn_01x10, Connector_JST:JST_GH_SM10B-GHS-TB_1x10-1MP_P1.25mm_Horizontal, B.Cu at (150.0, 121.5)
- added J3: Conn_01x10, Connector_JST:JST_GH_SM10B-GHS-TB_1x10-1MP_P1.25mm_Horizontal, B.Cu at (150.0, 78.6)
- added REF**: OSHW-Logo_11.4x12mm_Copper, Symbol:OSHW-Logo_11.4x12mm_Copper, B.Cu at (92.9, 119.1)
- moved SW72 45.4 mm to (150.0, 140.5)
- moved SW73 16.5 mm to (111.9, 140.5), turned to 0 degrees
Connections:
- D1 pad 1: GP4 -> GP5
- D10 pad 1: GP7 -> GP24
- D11 pad 1: GP8 -> GP29
- D12 pad 1: GP9 -> GP28
- D13 pad 1: GP4 -> GP5
- D14 pad 1: GP5 -> GP6
- D15 pad 1: GP6 -> GP23
- D16 pad 1: GP7 -> GP24
- D17 pad 1: GP8 -> GP29
- D18 pad 1: GP9 -> GP28
- D19 pad 1: GP6 -> GP23
- D2 pad 1: GP5 -> GP6
- D20 pad 1: GP7 -> GP24
- D21 pad 1: GP8 -> GP29
- D22 pad 1: GP9 -> GP28
- D3 pad 1: GP6 -> GP23
- D4 pad 1: GP7 -> GP24
- D5 pad 1: GP8 -> GP29
- D6 pad 1: GP9 -> GP28
- D7 pad 1: GP4 -> GP5
- D8 pad 1: GP5 -> GP6
- D9 pad 1: GP6 -> GP23
- MX1 pad 1: GP0 -> GP1
- MX10 pad 1: GP1 -> GP2
- MX11 pad 1: GP1 -> GP2
- MX12 pad 1: GP1 -> GP2
- MX13 pad 1: GP2 -> GP3
- MX14 pad 1: GP2 -> GP3
- MX15 pad 1: GP2 -> GP3
- MX16 pad 1: GP2 -> GP3
- MX17 pad 1: GP2 -> GP3
- MX18 pad 1: GP2 -> GP3
- MX19 pad 1: GP3 -> GP4
- MX2 pad 1: GP0 -> GP1
- MX20 pad 1: GP3 -> GP4
- MX21 pad 1: GP3 -> GP4
- MX22 pad 1: GP3 -> GP4
- MX3 pad 1: GP0 -> GP1
- MX4 pad 1: GP0 -> GP1
- MX45 pad 1: GP3 -> GP4
- MX5 pad 1: GP0 -> GP1
- MX6 pad 1: GP0 -> GP1
- MX7 pad 1: GP1 -> GP2
- MX8 pad 1: GP1 -> GP2
- MX9 pad 1: GP1 -> GP2
Routing:
- net GND: track 18.6 -> 185.0 mm, vias 16 -> 27
- net GP1: track 96.9 -> 226.5 mm, vias 0 -> 2
- net GP0: track 112.3 -> 0.00 mm
- net GP5: track 38.7 -> 150.1 mm, vias 0 -> 2
- net GP4: track 38.7 -> 141.1 mm
- net GP23: track 0.00 -> 99.9 mm, vias 0 -> 2
- net GP28: track 0.00 -> 94.0 mm, vias 0 -> 2
- net GP3: track 67.3 -> 153.1 mm, vias 0 -> 1
- net GP2: track 96.9 -> 178.7 mm, vias 0 -> 2
- net GP24: track 0.00 -> 75.3 mm, vias 0 -> 2
- net GP6: track 46.7 -> 121.4 mm, vias 0 -> 2
- net GP11: track 0.00 -> 66.6 mm, vias 0 -> 2
- net GP13: track 0.00 -> 66.4 mm, vias 0 -> 2
- net GP12: track 0.00 -> 66.3 mm, vias 0 -> 2
- net GP14: track 0.00 -> 65.9 mm, vias 0 -> 2
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- added copper zone on B.Cu, net +3.3V
Other:
- board text added: "1 2 3 4 5 6"
- board text added: "boot"
- board text added: "floookay.de/klappbrettle v1.0 — CERN-OHL-W"
- board text added: "reset"
